File: PCB/Cyberdeck Mech Keeb.brd (EAGLE design)
At the start: 262 x 110.5 mm, 86 parts, among them CN1 AUDIO-JACK3, CN2 AUDIO-JACK3, IC1 PCA9505, IC3 PCA9505, J1 SOLDERJUMPERTRACE, J2 SOLDERJUMPERTRACE, J3 SOLDERJUMPERTRACE, J5 SOLDERJUMPERTRACE, SW1 SPST_TACT-EVQQ2, SW10 KEYSWITCH-PLAIN-CHOC-1U, SW11 KEYSWITCH-PLAIN-CHOC-1U, SW12 KEYSWITCH-PLAIN-CHOC-1U, SW13 KEYSWITCH-PLAIN-CHOC-1U, SW14 KEYSWITCH-PLAIN-CHOC-1U, SW15 KEYSWITCH-PLAIN-CHOC-1U, SW16 KEYSWITCH-PLAIN-CHOC-1U, SW17 KEYSWITCH-PLAIN-CHOC-1U, SW18 KEYSWITCH-PLAIN-CHOC-1U, SW19 KEYSWITCH-PLAIN-CHOC-1U, SW2 SPST_TACT-EVQQ2, SW20 KEYSWITCH-PLAIN-CHOC-1U, SW21 KEYSWITCH-PLAIN-CHOC-1U, SW22 KEYSWITCH-PLAIN-CHOC-1U, SW23 KEYSWITCH-PLAIN-CHOC-1U, SW24 KEYSWITCH-PLAIN-CHOC-1U, SW25 KEYSWITCH-PLAIN-CHOC-1U, SW26 KEYSWITCH-PLAIN-CHOC-1U, SW27 KEYSWITCH-PLAIN-CHOC-1U, SW28 KEYSWITCH-PLAIN-CHOC-1U, SW29 KEYSWITCH-PLAIN-CHOC-1U, SW3 SPST_TACT-EVQQ2, SW30 KEYSWITCH-PLAIN-CHOC-1U, SW31 KEYSWITCH-PLAIN-CHOC-1U, SW32 KEYSWITCH-PLAIN-CHOC-1U, SW33 KEYSWITCH-PLAIN-CHOC-1U, SW34 KEYSWITCH-PLAIN-CHOC-1U, SW35 KEYSWITCH-PLAIN-CHOC-1U, SW36 KEYSWITCH-PLAIN-CHOC-1U, SW37 KEYSWITCH-PLAIN-CHOC-1U, SW38 KEYSWITCH-PLAIN-CHOC-1U, SW39 KEYSWITCH-PLAIN-CHOC-1U, SW4 SPST_TACT-EVQQ2, SW40 KEYSWITCH-PLAIN-CHOC-1U, SW41 KEYSWITCH-PLAIN-CHOC-1U, SW42 KEYSWITCH-PLAIN-CHOC-1U, SW43 KEYSWITCH-PLAIN-CHOC-1U, SW44 KEYSWITCH-PLAIN-CHOC-1U, SW45 KEYSWITCH-PLAIN-CHOC-1U, SW46 KEYSWITCH-PLAIN-CHOC-1U, SW47 KEYSWITCH-PLAIN-CHOC-1U, SW48 KEYSWITCH-PLAIN-CHOC-1U, SW49 KEYSWITCH-PLAIN-CHOC-1U, SW5 SPST_TACT-EVQQ2, SW50 KEYSWITCH-PLAIN-CHOC-1U, SW51 KEYSWITCH-PLAIN-CHOC-1U, SW52 KEYSWITCH-PLAIN-CHOC-1U, SW53 KEYSWITCH-PLAIN-CHOC-1U, SW54 KEYSWITCH-PLAIN-CHOC-1U, SW55 KEYSWITCH-PLAIN-CHOC-1U, SW56 KEYSWITCH-PLAIN-CHOC-1U, SW57 KEYSWITCH-PLAIN-CHOC-1U, SW58 KEYSWITCH-PLAIN-CHOC-1U, SW59 KEYSWITCH-PLAIN-CHOC-1U, SW6 SPST_TACT-EVQQ2, SW60 KEYSWITCH-PLAIN-CHOC-1U, SW61 KEYSWITCH-PLAIN-CHOC-1U, SW62 KEYSWITCH-PLAIN-CHOC-1U, SW63 KEYSWITCH-PLAIN-CHOC-1U, SW7 KEYSWITCH-PLAIN-CHOC-1U, SW8 KEYSWITCH-PLAIN-CHOC-1U, SW9 KEYSWITCH-PLAIN-CHOC-1U

Commit message: Gen 2 PCB
Parts:
- removed C22: 0.1uF, rcl:C0603
- removed J1, J2, J3, J5: SOLDERJUMPERTRACE, SparkFun-Passives:SJ_2S-TRACE
- removed JP3: (no value), pinhead:2X07
- removed MOD2, MOD3, MOD4: DISPLAY-OLED-128X64-I2C, diy-modules:DISPLAY-OLED-128X64-I2C
- removed SW3, SW4: SPST_TACT-EVQQ2, adafruit:EVQ-Q2
- added C1, C19, C2, C4, C5, C6: 0.1uF, rcl:C0603K
- added C10, C11, C12, C14, C15: 4.7uF, rcl:C0603K
- added C13, C7, C8, C9: 1uF, rcl:C0603K
- added C18: 4.7uF, adafruit:C0805
- added CN3, CN4: SATA, Voidstar-Connectors:SATA
- added D1, D2, D3: NVRB0530, adafruit:SOD-123FL
- added DISPLAY2: EINK-2.7, Voidstar-Silk:EINK-2.7
- added IC2, IC4, IC5: PCA9555D, micro-philips:SO24
- added IC6, IC7: 74HC30D, 74xx-eu:SO14
- added JP5, JP6: HEADER-0.1"-2.54MM-7POS, Voidstar-Connectors:2.54MM-7POS-SMD-RIGHTANGLE
- added L1: 10uH, Voidstar-Passive:CDRH6D12
- added Q1: SI1308EDL, SparkFun-DiscreteSemi:SOT323
- added R10, R12, R13, R14, R5, R6, R7, R8, R9: 10k, rcl:R0603
- added R11: 0.47, rcl:R0603
- added SJ1, SJ2: (no value), SparkFun-Passives:SJ_2
- added SW64, SW65, SW66, SW67, SW68, SW69_NICE, SW70, SW72, SW73: KEYSWITCH-MIRAGE-KITCHEN-SINK, Keyboard:CHOC-AND-MX-SOCKET-LED-MIRAGE-KITCHEN-SINK
- added X3: 52745-2490, con-molex:52745-2490
- added X4: 52745-0690, con-molex:52745-0690
- C16: value 0.1uF -> 1uF; device rcl:C0603 -> rcl:C0603K
- C17: value 0.1uF -> 4.7uF; device rcl:C0603 -> adafruit:C0805
- C3: device rcl:C0603 -> rcl:C0603K
- CN1, CN2: value AUDIO-JACK3 -> SATA; device SparkFun-Connectors:AUDIO-JACK-TRRS-SMD -> Voidstar-Connectors:SATA
- IC1, IC3: value PCA9505 -> PCA9555D; device micro-philips:TSSOP56-6 -> micro-philips:SO24
- JP1, JP2: value (none) -> HEADER-0.1"-2.54MM-7POS; device pinhead:1X04/90 -> Voidstar-Connectors:2.54MM-7POS-SMD-RIGHTANGLE
- R3, R4: value 4.7k -> 10k
- SW1, SW2, SW5, SW6: value SPST_TACT-EVQQ2 -> KEYSWITCH-MIRAGE-KITCHEN-SINK; device adafruit:EVQ-Q2 -> Keyboard:CHOC-AND-MX-SOCKET-LED-MIRAGE-KITCHEN-SINK
- SW10, SW11, SW12, SW13, SW14, SW15, SW16, SW17, SW18, SW19, SW20, SW21, SW22, SW23, SW24, SW25, SW26, SW27, SW28, SW29, SW30, SW31, SW32, SW33, SW34, SW35, SW36, SW37, SW38, SW39, SW40, SW41, SW42, SW43, SW44, SW45, SW46, SW47, SW48, SW49, SW50, SW51, SW52, SW53, SW54, SW55, SW56, SW57, SW58, SW59, SW60, SW61, SW62, SW63, SW7, SW8, SW9: value KEYSWITCH-PLAIN-CHOC-1U -> KEYSWITCH-MIRAGE-KITCHEN-SINK; device Keyboard:CHOC-1U -> Keyboard:CHOC-AND-MX-SOCKET-LED-MIRAGE-KITCHEN-SINK
- moved IC3 283.0 mm to (272.0, 107.2), flipped to the top, turned to 270 degrees
- moved C17 277.8 mm to (287.0, 65.0)
- moved C3 236.0 mm to (71.0, 114.0), flipped to the top, turned to 0 degrees
- moved SW6 228.1 mm to (39.2, 49.0), turned to 0 degrees
- moved CN1 197.5 mm to (18.0, 120.5), turned to 180 degrees
- moved IC1 193.1 mm to (120.0, 107.0), flipped to the top, turned to 270 degrees
- moved SW5 171.6 mm to (63.0, 11.0), turned to 0 degrees
- moved JP1 151.6 mm to (3.75, 103.0)
- moved C16 134.2 mm to (290.0, 69.5), turned to 90 degrees
- moved CN2 133.0 mm to (148.0, 120.5), turned to 180 degrees
- moved SW55 119.6 mm to (82.0, 11.0)
- moved SW62 119.6 mm to (272.0, 11.0)
- moved SW56 116.3 mm to (101.0, 11.0)
- moved SW57 113.2 mm to (124.8, 11.0)
- moved SW58 113.2 mm to (210.2, 11.0)
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Connections:
- removed net !INTERRUPT: IC1.55
- removed net !INTERRUPT': IC3.55
- removed net !RESET: IC1.56
- removed net !RESET': IC3.56
- removed net BAR: IC1.4, SW29.CHOC1
- removed net D10: JP3.8, MOD1.11
- removed net D2: JP3.5, MOD1.3
- removed net D3: JP3.7, MOD1.4
- removed net D8: JP3.12, MOD1.9
- removed net D9: JP3.10, MOD1.10
- removed net N$1: IC1.53, SW4.B
- removed net N$20: IC3.20, SW12.CHOC1
- removed net N$25: IC3.19, SW24.CHOC1
- removed net N$26: IC3.50, SW19.CHOC1
- removed net N$32: IC3.36, SW22.CHOC1
- removed net N$40: IC1.14, SW38.CHOC1
- removed net N$41: IC1.5, SW28.CHOC1
- removed net N$47: IC1.41, SW17.CHOC1
- removed net N$48: IC1.22, SW50.CHOC1
- removed net N$53: IC1.26, SW53.CHOC1
- removed net N$54: IC3.42, SW33.CHOC1
- removed net N$55: IC1.40, SW16.CHOC1
- removed net N$6: IC3.10, SW9.CHOC1
- removed net N$7: IC1.7, SW27.CHOC1
- removed net N$74: IC3.53, SW43.CHOC1
- removed net N$75: IC3.24, SW37.CHOC1
- removed net N$78: IC3.43, SW45.CHOC1
- removed net N$80: IC3.38, SW46.CHOC1
- removed net N$82: IC3.32, SW47.CHOC1
- removed net N$86: IC3.21, SW61.CHOC1
- removed net SCL2: JP3.13, MOD1.8, MOD4.3, R4.1
- removed net SDA2: JP3.14, MOD1.7, MOD4.4, R3.1
- removed net VCC/2: C17.1, C22.1, CN2.TIP, IC3.11, IC3.23, IC3.27, IC3.28, IC3.34, IC3.39, IC3.51, IC3.6, J5.1, JP2.4
- removed net VIN: JP3.2, MOD1.14
- new net +5V: CN3.P$6, CN4.P$6, JP5.2, JP6.6, MOD1.14, SW1.+1, SW13.+1, SW14.+1, SW15.+1, SW16.+1, SW17.+1, SW18.+1, SW2.+1, SW25.+1, SW26.+1, SW27.+1, SW28.+1, SW29.+1, SW30.+1, SW37.+1, SW38.+1, SW39.+1, SW40.+1, SW41.+1, SW42.+1, SW49.+1, SW50.+1, SW51.+1, SW52.+1, SW53.+1, SW54.+1, SW58.+1, SW59.+1, SW60.+1, SW61.+1, SW62.+1
- new net +5V/2: CN1.P$6, CN2.P$6, JP1.2, JP2.6, SW10.+1, SW11.+1, SW12.+1, SW19.+1, SW20.+1, SW21.+1, SW22.+1, SW23.+1, SW24.+1, SW31.+1, SW32.+1, SW33.+1, SW34.+1, SW35.+1, SW36.+1, SW43.+1, SW44.+1, SW45.+1, SW46.+1, SW47.+1, SW48.+1, SW5.+1, SW55.+1, SW56.+1, SW57.+1, SW6.+1, SW63.+1, SW64.+1, SW65.+1, SW66.+1, SW67.+1, SW68.+1, SW69_NICE.+1, SW7.+1, SW70.+1, SW72.+1, SW73.+1, SW8.+1, SW9.+1
- new net COL10LED: SW15.DI1, SW16.DO1
- new net COL11LED: SW59.DI1, SW60.DO1
- new net COL12LED: SW17.DI1, SW18.DO1
- new net COL13LED: SW2.DO1, SW62.DI1
- new net COL1LED: SW72.DI1, SW73.DO1
- new net COL2LED: SW65.DI1, SW7.DO1
- new net COL3LED: SW5.DI1, SW55.DO1
- new net COL4LED: SW8.DI1, SW9.DO1
- new net COL5LED: SW46.DO1, SW56.DI1
- new net COL6LED: SW10.DI1, SW11.DO1
- new net COL7LED: SW57.DI1, SW63.DO1
- new net COL8LED: SW13.DI1, SW14.DO1
- new net COL9LED: SW50.DI1, SW58.DO1
- new net D6: MOD1.7
- new net DISPLAY_BUSY: MOD1.10, X3.16
- new net DISPLAY_RESET: IC3.20, R13.1, X3.15, X4.4
- new net EXPANDER0_INT: IC4.1, IC7.4, R7.1
- new net EXPANDER1_INT: IC2.1, IC7.5, R6.1
- new net EXPANDER2_INT: IC1.1, IC7.6, R5.1
- new net EXPANDER3_INT: IC5.1, IC6.6, R10.1
- new net EXPANDER4_INT: IC3.1, IC6.1, R3.1
- new net GDR: Q1.1, R9.2, X3.23
- new net INTERRUPT: IC6.8, MOD1.4, R4.2
- new net LEFTER_HAND_INT: CN1.P$4, IC7.3, JP1.4
- new net LEFTER_HAND_LED: CN1.P$3, JP1.5, SW66.DO1
- new net LEFT_HAND_INT: CN3.P$4, IC6.2, JP5.4
- new net LEFT_HAND_INT': CN2.P$4, IC7.8, JP2.4, R14.2
- new net LEFT_HAND_LED: CN3.P$3, JP5.5, SW61.DO1
- new net LEFT_HAND_LED': CN2.P$3, JP2.3, SW12.DI1
- new net N$107: IC4.18
- new net N$109: IC4.20
- new net N$128: IC2.4
- new net N$129: IC2.5
- new net N$149: SW53.DO1, SW60.DI1
- new net N$150: SW41.DO1, SW53.DI1
- new net N$151: SW29.DO1, SW41.DI1
- new net N$152: SW17.DO1, SW29.DI1
- new net N$154: SW1.DO1, SW2.DI1
- new net N$163: SW15.DO1, SW27.DI1
- new net N$164: SW27.DO1, SW39.DI1
- new net N$165: SW39.DO1, SW51.DI1
- new net N$166: SW51.DO1, SW58.DI1
- new net N$18: SW11.DI1, SW23.DO1
- new net N$45: SW32.DO1, SW44.DI1
- new net N$58: SW6.DO1, SW69_NICE.DI1
- new net N$59: SW69_NICE.DO1, SW73.DI1
- new net N$61: IC4.15
- new net N$62: IC4.16
- new net N$65: SW64.DI1, SW70.DO1
- new net N$66: SW64.DO1, SW66.DI1
- new net PREVGH: C16.2, D1.C, X3.4
- new net PREVGL: C12.2, D3.A, X3.2
- new net QUAGSIRE: IC2.6
- new net R0C0: IC4.4, SW66.CHOC2, SW66.MX2
- new net R0C1: IC4.11, SW65.CHOC1, SW65.MX1
- new net R0C10: IC5.15, SW15.CHOC2, SW15.MX2
- new net R0C11: IC5.19, SW16.CHOC1, SW16.MX1
- new net R0C12: IC3.7, SW17.CHOC2, SW17.MX2
- new net R0C13: IC3.13, SW18.CHOC2, SW18.MX2
- new net R0C2: IC2.11, SW7.CHOC1, SW7.MX1
- new net R0C3: IC2.17, SW8.CHOC1, SW8.MX1
- new net R0C4: IC1.4, SW9.CHOC1, SW9.MX1
- new net R0C5: IC1.9, SW10.CHOC1, SW10.MX1
- new net R0C6: IC1.15, SW11.CHOC1, SW11.MX1
- new net R0C7: IC1.20, SW12.CHOC1, SW12.MX1
- new net R0C8: IC5.4, SW13.CHOC2, SW13.MX2
- new net R0C9: IC5.9, SW14.CHOC2, SW14.MX2
- new net R1C0: IC4.5, SW64.CHOC2, SW64.MX2
- new net R1C1: IC4.10, SW67.CHOC1, SW67.MX1
- new net R1C10: IC5.16, SW27.CHOC2, SW27.MX2
- new net R1C11: IC5.20, SW28.CHOC2, SW28.MX2
- new net R1C12: IC3.8, SW29.CHOC2, SW29.MX2
- new net R1C13: IC3.14, SW30.CHOC2, SW30.MX2
- new net R1C2: IC2.10, SW19.CHOC1, SW19.MX1
- new net R1C3: IC2.16, SW20.CHOC1, SW20.MX1
- new net R1C4: IC2.20, SW21.CHOC1, SW21.MX1
- new net R1C5: IC1.8, SW22.CHOC1, SW22.MX1
- new net R1C6: IC1.14, SW23.CHOC1, SW23.MX1
- new net R1C7: IC1.19, SW24.CHOC1, SW24.MX1
- new net R1C8: IC5.5, SW25.CHOC2, SW25.MX2
- new net R1C9: IC5.10, SW26.CHOC2, SW26.MX2
- new net R2C0: IC4.6, SW70.CHOC2, SW70.MX2
- new net R2C1: IC4.9, SW6.CHOC1, SW6.MX1
- new net R2C10: IC5.17, SW39.CHOC2, SW39.MX2
- new net R2C11: IC3.4, SW40.CHOC2, SW40.MX2
- new net R2C12: IC3.9, SW41.CHOC2, SW41.MX2
- new net R2C13: IC3.15, SW42.CHOC2, SW42.MX2
- new net R2C2: IC2.9, SW31.CHOC1, SW31.MX1
- new net R2C3: IC2.15, SW32.CHOC1, SW32.MX1
- new net R2C4: IC2.19, SW33.CHOC1, SW33.MX1
- new net R2C5: IC1.7, SW34.CHOC1, SW34.MX1
- new net R2C6: IC1.13, SW35.CHOC1, SW35.MX1
- new net R2C7: IC1.18, SW36.CHOC1, SW36.MX1
- new net R2C8: IC5.6, SW37.CHOC2, SW37.MX2
- new net R2C9: IC5.11, SW38.CHOC2, SW38.MX2
- new net R3C0: IC4.7, SW68.CHOC2, SW68.MX2
- new net R3C1: IC4.13, SW69_NICE.CHOC2, SW69_NICE.MX2
- new net R3C10: IC5.18, SW51.CHOC2, SW51.MX2
- new net R3C11: IC3.5, SW52.CHOC2, SW52.MX2
- new net R3C12: IC3.10, SW53.CHOC2, SW53.MX2
- new net R3C13: IC3.16, SW54.CHOC2, SW54.MX2
- new net R3C2: IC2.8, SW43.CHOC1, SW43.MX1
- new net R3C3: IC2.14, SW44.CHOC1, SW44.MX1
- new net R3C4: IC2.18, SW45.CHOC1, SW45.MX1
- new net R3C5: IC1.6, SW46.CHOC1, SW46.MX1
- new net R3C6: IC1.10, SW47.CHOC1, SW47.MX1
- new net R3C7: IC1.17, SW48.CHOC1, SW48.MX1
- new net R3C8: IC5.7, SW49.CHOC2, SW49.MX2
- new net R3C9: IC5.14, SW50.CHOC2, SW50.MX2
- new net R4C0: IC4.8, SW72.CHOC2, SW72.MX2
- new net R4C1: IC4.14, SW73.CHOC2, SW73.MX2
- new net R4C10: IC5.13, SW58.CHOC1, SW58.MX1
- new net R4C11: IC3.6, SW59.CHOC2, SW59.MX2
- new net R4C12: IC3.11, SW60.CHOC2, SW60.MX2
- new net R4C13: IC3.17, SW62.CHOC2, SW62.MX2
- new net R4C14: IC3.18, SW2.CHOC1, SW2.MX1
- new net R4C15: IC3.19, SW1.CHOC2, SW1.MX2
- new net R4C2: IC2.7, SW5.CHOC1, SW5.MX1
- new net R4C3: IC2.13, SW55.CHOC1, SW55.MX1
- new net R4C4: IC1.5, SW56.CHOC2, SW56.MX2
- new net R4C6: IC1.11, SW57.CHOC2, SW57.MX2
- new net R4C7: IC1.16, SW63.CHOC1, SW63.MX1
- new net R4C8: IC5.8, SW61.CHOC2, SW61.MX2
- new net RAGE_LEDS: MOD1.8, SW1.DI1
- new net RESE: Q1.2, R11.2, X3.22
- new net RIGHTER_HAND_INT: CN4.P$4, IC6.11, JP6.4
- new net RIGHTER_HAND_LED: CN4.P$3, JP6.3, MOD1.3
- new net SCK: MOD1.9, X3.12
- new net SDI: MOD1.11, X3.11
- new net THIRD_HALF_SELECT: IC1.21, IC2.21, IC4.21, R8.1, SJ1.2, SJ2.2
- new net THIS_IS_LEFTER: IC4.19, SJ2.1
- new net THIS_IS_RIGHTER: IC4.17, SJ2.3
- new net TOUCH_INT: IC6.12, R12.1, X4.5
- new net TSCL: X3.19
- new net TSDA: X3.18
- new net VCCIO: C1.1, C19.1, C2.1, C3.1, CN1.P$7, CN2.P$7, IC1.2, IC1.24, IC2.2, IC2.24, IC2.3, IC4.24, IC7.14, JP1.1, JP2.7, R5.2, R6.2, R7.2, R8.2, SJ1.3
- new net VCOM: C13.2, X3.1
- new net VDD: C8.2, X3.7
- new net VGH: C15.2, X3.20
- new net VGL: C14.2, X3.21
- new net VPP: C9.2, X3.6
- new net VSH: C10.2, X3.5
- new net VSL: C11.2, X3.3
- net +3V3: now also C18.1, C4.1, C5.1, C6.1, C7.2, CN3.P$7, CN4.P$7, IC3.21, IC3.24, IC3.3, IC5.24, IC5.3, IC6.14, JP5.1, JP6.7, L1.P$1, R10.2, R12.2, R13.2, X3.10, X3.17, X3.9, X4.3; no longer C16.1, C3.1, CN1.TIP, IC1.11, IC1.23, IC1.27, IC1.28, IC1.29, IC1.34, IC1.39, IC1.51, IC1.6, J5.2, JP1.1, JP3.6, MOD2.2, MOD3.2, MOD4.2, R4.2
- net D0: no longer JP3.1
- net D1: no longer JP3.3
- net GND: now also C10.1, C11.1, C12.1, C13.1, C14.1, C15.1, C16.1, C18.2, C4.2, C5.2, C6.2, C7.1, C8.1, C9.1, CN3.LEFT_TAB, CN3.P$5, CN3.RIGHT_TAB, CN4.LEFT_TAB, CN4.P$5, CN4.RIGHT_TAB, D2.C, IC3.12, IC3.2, IC5.12, IC5.2, IC5.21, IC6.7, JP5.3, JP6.5, R11.1, R4.1, R9.1, SW1.CHOC1, SW1.GND1, SW1.MX1, SW13.CHOC1, SW13.GND1, SW13.MX1, SW14.CHOC1, SW14.GND1, SW14.MX1, SW15.CHOC1, SW15.GND1, SW15.MX1, SW16.GND1, SW16.MX2, SW17.CHOC1, SW17.GND1, SW17.MX1, SW18.CHOC1, SW18.GND1, SW18.MX1, SW2.CHOC2, SW2.GND1, SW2.MX2, SW25.CHOC1, SW25.GND1, SW25.MX1, SW26.CHOC1, SW26.GND1, SW26.MX1, SW27.CHOC1, SW27.GND1, SW27.MX1, SW28.CHOC1, SW28.GND1, SW28.MX1, SW29.CHOC1, SW29.GND1, SW29.MX1, SW30.CHOC1, SW30.GND1, SW30.MX1, SW37.CHOC1, SW37.GND1, SW37.MX1, SW38.CHOC1, SW38.GND1, SW38.MX1, SW39.CHOC1, SW39.GND1, SW39.MX1, SW40.CHOC1, SW40.GND1, SW40.MX1, SW41.CHOC1, SW41.GND1, SW41.MX1, SW42.CHOC1, SW42.GND1, SW42.MX1, SW49.CHOC1, SW49.GND1, SW49.MX1, SW50.CHOC1, SW50.GND1, SW50.MX1, SW51.CHOC1, SW51.GND1, SW51.MX1, SW52.CHOC1, SW52.GND1, SW52.MX1, SW53.CHOC1, SW53.GND1, SW53.MX1, SW54.CHOC1, SW54.GND1, SW54.MX1, SW58.GND1, SW58.MX2, SW59.CHOC1, SW59.GND1, SW59.MX1, SW60.CHOC1, SW60.GND1, SW60.MX1, SW61.CHOC1, SW61.GND1, SW61.MX1, SW62.CHOC1, SW62.GND1, SW62.MX1, X3.13, X3.14, X3.8, X4.6; no longer C16.2, C3.2, CN1.EARTH, IC1.18, IC1.30, IC1.46, J1.2, JP1.4, JP3.4, MOD2.1, MOD3.1, MOD4.1, SW1.A, SW14.CHOC2, SW15.CHOC2, SW17.CHOC2, SW18.CHOC2, SW2.A, SW26.CHOC2, SW27.CHOC2, SW28.CHOC2, SW29.CHOC2, SW3.A, SW30.CHOC2, SW38.CHOC2, SW39.CHOC2, SW4.A, SW40.CHOC2, SW41.CHOC2, SW42.CHOC2, SW5.A, SW50.CHOC2, SW51.CHOC2, SW52.CHOC2, SW53.CHOC2, SW54.CHOC2, SW59.CHOC2, SW6.A, SW60.CHOC2, SW62.CHOC2
- net GND2: now also C1.2, C19.2, C2.2, C3.2, CN1.LEFT_TAB, CN1.P$5, CN1.RIGHT_TAB, CN2.LEFT_TAB, CN2.P$5, CN2.RIGHT_TAB, IC1.12, IC1.3, IC2.12, IC4.12, IC4.2, IC4.3, IC7.7, JP1.3, JP2.5, R14.1, SJ1.1, SW10.GND1, SW10.MX2, SW11.GND1, SW11.MX2, SW12.GND1, SW12.MX2, SW19.GND1, SW19.MX2, SW20.GND1, SW20.MX2, SW21.GND1, SW21.MX2, SW22.GND1, SW22.MX2, SW23.GND1, SW23.MX2, SW24.GND1, SW24.MX2, SW31.GND1, SW31.MX2, SW32.GND1, SW32.MX2, SW33.GND1, SW33.MX2, SW34.GND1, SW34.MX2, SW35.GND1, SW35.MX2, SW36.GND1, SW36.MX2, SW43.GND1, SW43.MX2, SW44.GND1, SW44.MX2, SW45.GND1, SW45.MX2, SW46.GND1, SW46.MX2, SW47.GND1, SW47.MX2, SW48.GND1, SW48.MX2, SW5.CHOC2, SW5.GND1, SW5.MX2, SW55.GND1, SW55.MX2, SW56.CHOC1, SW56.GND1, SW56.MX1, SW57.CHOC1, SW57.GND1, SW57.MX1, SW6.CHOC2, SW6.GND1, SW6.MX2, SW63.GND1, SW63.MX2, SW64.CHOC1, SW64.GND1, SW64.MX1, SW65.CHOC2, SW65.GND1, SW65.MX2, SW66.CHOC1, SW66.GND1, SW66.MX1, SW67.CHOC2, SW67.GND1, SW67.MX2, SW68.CHOC1, SW68.GND1, SW68.MX1, SW69_NICE.CHOC1, SW69_NICE.GND1, SW69_NICE.MX1, SW7.GND1, SW7.MX2, SW70.CHOC1, SW70.GND1, SW70.MX1, SW72.CHOC1, SW72.GND1, SW72.MX1, SW73.CHOC1, SW73.GND1, SW73.MX1, SW8.GND1, SW8.MX2, SW9.GND1, SW9.MX2; no longer C17.2, C22.2, CN2.EARTH, IC3.18, IC3.29, IC3.30, IC3.46, J1.1, JP2.1, SW13.CHOC2, SW25.CHOC2, SW37.CHOC2, SW49.CHOC2, SW56.CHOC2, SW57.CHOC2, SW61.CHOC2
- net N$10: now also SW25.DO1, SW37.DI1; no longer IC1.21, SW58.CHOC1
- net N$11: now also C17.1, D2.A, D3.C; no longer IC1.42, SW18.CHOC1
- net N$12: now also SW35.DI1, SW47.DO1; no longer IC3.47, SW32.CHOC1
- net N$13: now also SW37.DO1, SW49.DI1; no longer IC3.22, SW49.CHOC1
- net N$14: now also SW23.DI1, SW35.DO1; no longer IC3.49, SW44.CHOC1
- net N$15: now also SW42.DI1, SW54.DO1; no longer IC1.8, SW26.CHOC1
- net N$16: now also SW54.DI1, SW62.DO1; no longer IC1.37, SW14.CHOC1
- net N$17: now also C17.2, D1.A, L1.P$3, Q1.3; no longer IC1.3, SW30.CHOC1
- net N$19: now also SW30.DI1, SW42.DO1; no longer IC3.35, SW57.CHOC1
- net N$2: now also SW12.DO1, SW24.DI1; no longer IC3.48, SW7.CHOC1
- net N$21: now also SW18.DI1, SW30.DO1; no longer IC3.44, SW56.CHOC1
- net N$22: now also SW14.DI1, SW26.DO1; no longer IC1.15, SW54.CHOC1
- net N$23: now also SW16.DI1, SW28.DO1; no longer IC3.54, SW55.CHOC1
- net N$24: now also SW28.DI1, SW40.DO1; no longer IC1.9, SW42.CHOC1
- net N$27: now also SW10.DO1, SW22.DI1; no longer IC1.43, SW1.B
- net N$28: now also SW22.DO1, SW34.DI1; no longer IC3.45, SW20.CHOC1
- net N$29: now also SW40.DI1, SW52.DO1; no longer IC1.13, SW39.CHOC1
- net N$3: now also SW24.DO1, SW36.DI1; no longer IC1.45, SW5.B
- net N$30: now also SW34.DO1, SW46.DI1; no longer IC3.41, SW21.CHOC1
- net N$31: now also SW52.DI1, SW59.DO1; no longer IC1.19, SW62.CHOC1
- net N$33: now also SW26.DI1, SW38.DO1; no longer IC1.12, SW40.CHOC1
- net N$34: now also SW38.DI1, SW50.DO1; no longer IC3.26, SW13.CHOC1
- net N$35: now also SW45.DI1, SW56.DO1; no longer IC3.17, SW36.CHOC1
- net N$36: now also SW33.DI1, SW45.DO1; no longer IC3.13, SW35.CHOC1
- net N$37: now also SW49.DO1, SW61.DI1; no longer IC1.16, SW60.CHOC1
- net N$38: now also SW21.DI1, SW33.DO1; no longer IC3.16, SW48.CHOC1
- net N$39: now also SW21.DO1, SW9.DI1; no longer IC1.20, SW59.CHOC1
- net N$4: now also SW36.DO1, SW48.DI1; no longer IC3.9, SW8.CHOC1
- net N$43: now also SW20.DI1, SW8.DO1; no longer IC3.14, SW23.CHOC1
- net N$44: now also SW20.DO1, SW32.DI1; no longer IC3.15, SW11.CHOC1
- net N$46: now also SW44.DO1, SW55.DI1; no longer IC1.54, SW6.B'
- net N$49: now also SW43.DI1, SW5.DO1; no longer IC1.24, SW51.CHOC1
- net N$5: now also SW48.DO1, SW63.DI1; no longer IC1.52, SW2.B
- net N$50: now also SW31.DI1, SW43.DO1; no longer IC3.52, SW31.CHOC1
- net N$51: now also SW19.DI1, SW31.DO1; no longer IC1.25, SW52.CHOC1
- net N$52: now also SW19.DO1, SW7.DI1; no longer IC1.44, SW3.B
- net N$56: now also SW65.DO1, SW67.DI1; no longer IC3.37, SW34.CHOC1
- net N$57: now also SW6.DI1, SW67.DO1; no longer IC3.33, SW63.CHOC1
- net N$63: now also SW68.DI1, SW72.DO1; no longer IC1.38, SW15.CHOC1
- net N$64: now also SW68.DO1, SW70.DI1; no longer IC1.10, SW41.CHOC1
- net N$8: now also SW47.DI1, SW57.DO1; no longer IC3.12, SW10.CHOC1
- net N$9: now also SW13.DO1, SW25.DI1; no longer IC3.25, SW25.CHOC1
- net SCL: now also CN3.P$1, CN4.P$1, IC3.22, IC5.22, JP5.7, JP6.1, X4.2; no longer CN1.RING1, IC1.2, J3.2, JP1.2, JP3.11, MOD2.3, MOD3.3
- net SCL': now also CN1.P$1, CN2.P$1, IC1.22, IC2.22, IC4.22, JP1.7, JP2.1; no longer CN2.RING1, IC3.2, J3.1, JP2.3
- net SDA: now also CN3.P$2, CN4.P$2, IC3.23, IC5.23, JP5.6, JP6.2, X4.1; no longer CN1.RING2, IC1.1, J2.2, JP1.3, JP3.9, MOD2.4, MOD3.4
- net SDA': now also CN1.P$2, CN2.P$2, IC1.23, IC2.23, IC4.23, JP1.6; no longer CN2.RING2, IC3.1, J2.1
Routing:
- net +5V/2: track 0.00 -> 1189.0 mm, vias 0 -> 49
- net +5V: track 0.00 -> 1138.9 mm, vias 0 -> 31
- net +3V3: track 376.9 -> 745.6 mm, vias 22 -> 16
- net VCCIO: track 0.00 -> 356.0 mm, vias 0 -> 17
- net N$86: track 179.5 -> 0.00 mm
- net VCC/2: track 170.3 -> 0.00 mm, vias 6 -> 0
- net RAGE_LEDS: track 0.00 -> 160.5 mm, vias 0 -> 2
- net SDA2: track 143.8 -> 0.00 mm, vias 4 -> 0
- net R4C15: track 0.00 -> 143.6 mm, vias 0 -> 1
- net N$75: track 142.3 -> 0.00 mm
- net SCL2: track 141.2 -> 0.00 mm, vias 6 -> 0
- net N$13: track 161.8 -> 23.6 mm
- net LEFTER_HAND_INT: track 0.00 -> 137.9 mm, vias 0 -> 2
- net RIGHTER_HAND_LED: track 0.00 -> 132.6 mm, vias 0 -> 3
- net RIGHTER_HAND_INT: track 0.00 -> 127.2 mm, vias 0 -> 2
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Other:
- board size 262 x 110.5 mm -> 335 x 201.8 mm
- board text added: "(c) 2021 Voidstar Lab LEFT HAND PROTOTYPE v2 PRINTING A (That one time I only fabbed the left hand)"
- board text added: "(c) 2021 Voidstar Lab RIGHT HAND PROTOTYPE v2 PRINTING A (That one time I only fabbed the right hand)"
- board text added: "...and it's on"
- board text added: "If the project is done, just add another half. There is no escape."
- board text added: "This is the"
- board text added: "left board"
- board text added: "the left side"
- board text added: "the right side"
- board text added: "third board"
- board text removed: "(c) 2021 Voidstar Lab"
- board text removed: "(c) 2021 Voidstar Lab LLC LEFT HAND PROTOTYPE v1 PRINTING A"
- board text removed: "(c) 2021 Voidstar Lab RIGHT HAND PROTOTYPE v1 PRINTING A"
- board text removed: "9x MILLED SLOTS 1mm WIDE"
- board text removed: "BOARD"
- board text removed: "BOARDS BY"
- board text removed: "CHOC SPACING SHOULD BE 18x17 NOT 19x19"
- board text removed: "DECK"
- board text removed: "IN PARTNERSHIP WITH"
- board text removed: "If the project is half done, just delete the other half. Now your project is done."
- board text removed: "KEYBOARD"
- board text removed: "LAB"
- board text removed: "MI"
- board text removed: "MIRAG"
- board text removed: "NEXTPCB"
- board text removed: "ONE HALF IS A MACRO PAD AND"
- board text removed: "Pads should be longer"
- board text removed: "RAGE"
- board text removed: "THREE HALVES A CYBER"
- board text removed: "VOIDSTAR"
- board text removed: "ZACK FREEDMAN of VOIDSTAR LAB"
- board text removed: "proudly presents the"
