File: PCB/Cyberdeck Mech Keeb.sch (EAGLE design)
At the start: 86 parts, among them CN1 AUDIO-JACK3, CN2 AUDIO-JACK3, IC1 PCA9505, IC3 PCA9505, J1 SOLDERJUMPERTRACE, J2 SOLDERJUMPERTRACE, J3 SOLDERJUMPERTRACE, J5 SOLDERJUMPERTRACE, SW1 SPST_TACT-EVQQ2, SW10 KEYSWITCH-PLAIN-CHOC-1U, SW11 KEYSWITCH-PLAIN-CHOC-1U, SW12 KEYSWITCH-PLAIN-CHOC-1U, SW13 KEYSWITCH-PLAIN-CHOC-1U, SW14 KEYSWITCH-PLAIN-CHOC-1U, SW15 KEYSWITCH-PLAIN-CHOC-1U, SW16 KEYSWITCH-PLAIN-CHOC-1U, SW17 KEYSWITCH-PLAIN-CHOC-1U, SW18 KEYSWITCH-PLAIN-CHOC-1U, SW19 KEYSWITCH-PLAIN-CHOC-1U, SW2 SPST_TACT-EVQQ2, SW20 KEYSWITCH-PLAIN-CHOC-1U, SW21 KEYSWITCH-PLAIN-CHOC-1U, SW22 KEYSWITCH-PLAIN-CHOC-1U, SW23 KEYSWITCH-PLAIN-CHOC-1U, SW24 KEYSWITCH-PLAIN-CHOC-1U, SW25 KEYSWITCH-PLAIN-CHOC-1U, SW26 KEYSWITCH-PLAIN-CHOC-1U, SW27 KEYSWITCH-PLAIN-CHOC-1U, SW28 KEYSWITCH-PLAIN-CHOC-1U, SW29 KEYSWITCH-PLAIN-CHOC-1U, SW3 SPST_TACT-EVQQ2, SW30 KEYSWITCH-PLAIN-CHOC-1U, SW31 KEYSWITCH-PLAIN-CHOC-1U, SW32 KEYSWITCH-PLAIN-CHOC-1U, SW33 KEYSWITCH-PLAIN-CHOC-1U, SW34 KEYSWITCH-PLAIN-CHOC-1U, SW35 KEYSWITCH-PLAIN-CHOC-1U, SW36 KEYSWITCH-PLAIN-CHOC-1U, SW37 KEYSWITCH-PLAIN-CHOC-1U, SW38 KEYSWITCH-PLAIN-CHOC-1U, SW39 KEYSWITCH-PLAIN-CHOC-1U, SW4 SPST_TACT-EVQQ2, SW40 KEYSWITCH-PLAIN-CHOC-1U, SW41 KEYSWITCH-PLAIN-CHOC-1U, SW42 KEYSWITCH-PLAIN-CHOC-1U, SW43 KEYSWITCH-PLAIN-CHOC-1U, SW44 KEYSWITCH-PLAIN-CHOC-1U, SW45 KEYSWITCH-PLAIN-CHOC-1U, SW46 KEYSWITCH-PLAIN-CHOC-1U, SW47 KEYSWITCH-PLAIN-CHOC-1U, SW48 KEYSWITCH-PLAIN-CHOC-1U, SW49 KEYSWITCH-PLAIN-CHOC-1U, SW5 SPST_TACT-EVQQ2, SW50 KEYSWITCH-PLAIN-CHOC-1U, SW51 KEYSWITCH-PLAIN-CHOC-1U, SW52 KEYSWITCH-PLAIN-CHOC-1U, SW53 KEYSWITCH-PLAIN-CHOC-1U, SW54 KEYSWITCH-PLAIN-CHOC-1U, SW55 KEYSWITCH-PLAIN-CHOC-1U, SW56 KEYSWITCH-PLAIN-CHOC-1U, SW57 KEYSWITCH-PLAIN-CHOC-1U, SW58 KEYSWITCH-PLAIN-CHOC-1U, SW59 KEYSWITCH-PLAIN-CHOC-1U, SW6 SPST_TACT-EVQQ2, SW60 KEYSWITCH-PLAIN-CHOC-1U, SW61 KEYSWITCH-PLAIN-CHOC-1U, SW62 KEYSWITCH-PLAIN-CHOC-1U, SW63 KEYSWITCH-PLAIN-CHOC-1U, SW7 KEYSWITCH-PLAIN-CHOC-1U, SW8 KEYSWITCH-PLAIN-CHOC-1U, SW9 KEYSWITCH-PLAIN-CHOC-1U

Commit message: Gen 2 PCB
Parts:
- removed C22: 0.1uF, rcl:C-USC0603
- removed J1, J2, J3, J5: SOLDERJUMPERTRACE, SparkFun-Passives:SOLDERJUMPERTRACE
- removed JP3: (no value), pinhead:PINHD-2X7
- removed MOD2, MOD3, MOD4: DISPLAY-OLED-128X64-I2C, diy-modules:DISPLAY-OLED-128X64-I2C
- removed SW3, SW4: SPST_TACT-EVQQ2, adafruit:SPST_TACT-EVQQ2
- added C1, C19, C2, C4, C5, C6: 0.1uF, rcl:C-USC0603K
- added C10, C11, C12, C14, C15: 4.7uF, rcl:C-USC0603K
- added C13, C7, C8, C9: 1uF, rcl:C-USC0603K
- added C18: 4.7uF, adafruit:C-USC0805
- added CN3, CN4: SATA, Voidstar-Connectors:SATA
- added D1, D2, D3: NVRB0530, adafruit:DIODE_SOD-123FL
- added DISPLAY2: EINK-2.7, Voidstar-Silk:EINK-2.7
- added IC2, IC4, IC5: PCA9555D, micro-philips:PCA9555D
- added IC6, IC7: 74HC30D, 74xx-eu:74HC30D
- added JP5, JP6: HEADER-0.1"-2.54MM-7POS, Voidstar-Connectors:HEADER-0.1"-2.54MM-7POS
- added L1: 10uH, Voidstar-Passive:CDRH6D12
- added Q1: SI1308EDL, SparkFun-DiscreteSemi:MOSFET-NCHANNEL2N7002PW
- added R10, R12, R13, R14, R5, R6, R7, R8, R9: 10k, rcl:R-US_R0603
- added R11: 0.47, rcl:R-US_R0603
- added SJ1, SJ2: (no value), SparkFun-Passives:SOLDERJUMPER_2WAYT
- added SW64, SW65, SW66, SW67, SW68, SW69_NICE, SW70, SW72, SW73: KEYSWITCH-MIRAGE-KITCHEN-SINK, Keyboard:KEYSWITCH-MIRAGE-KITCHEN-SINK
- added X3: 52745-2490, con-molex:52745-2490
- added X4: 52745-0690, con-molex:52745-0690
- C16: value 0.1uF -> 1uF; device rcl:C-USC0603 -> rcl:C-USC0603K
- C17: value 0.1uF -> 4.7uF; device rcl:C-USC0603 -> adafruit:C-USC0805
- C3: device rcl:C-USC0603 -> rcl:C-USC0603K
- CN1, CN2: value AUDIO-JACK3 -> SATA; device SparkFun-Connectors:AUDIO-JACK3 -> Voidstar-Connectors:SATA
- IC1, IC3: value PCA9505 -> PCA9555D; device micro-philips:PCA9505 -> micro-philips:PCA9555D
- JP1, JP2: value (none) -> HEADER-0.1"-2.54MM-7POS; device pinhead:PINHD-1X4/90 -> Voidstar-Connectors:HEADER-0.1"-2.54MM-7POS
- R3, R4: value 4.7k -> 10k
- SW1, SW2, SW5, SW6: value SPST_TACT-EVQQ2 -> KEYSWITCH-MIRAGE-KITCHEN-SINK; device adafruit:SPST_TACT-EVQQ2 -> Keyboard:KEYSWITCH-MIRAGE-KITCHEN-SINK
- SW10, SW11, SW12, SW13, SW14, SW15, SW16, SW17, SW18, SW19, SW20, SW21, SW22, SW23, SW24, SW25, SW26, SW27, SW28, SW29, SW30, SW31, SW32, SW33, SW34, SW35, SW36, SW37, SW38, SW39, SW40, SW41, SW42, SW43, SW44, SW45, SW46, SW47, SW48, SW49, SW50, SW51, SW52, SW53, SW54, SW55, SW56, SW57, SW58, SW59, SW60, SW61, SW62, SW63, SW7, SW8, SW9: value KEYSWITCH-PLAIN-CHOC-1U -> KEYSWITCH-MIRAGE-KITCHEN-SINK; device Keyboard:KEYSWITCH-PLAIN-CHOC-1U -> Keyboard:KEYSWITCH-MIRAGE-KITCHEN-SINK
Connections:
- removed net !INTERRUPT: IC1.!INT
- removed net !INTERRUPT': IC3.!INT
- removed net !RESET: IC1.!RESET
- removed net !RESET': IC3.!RESET
- removed net BAR: IC1.IO0_1, SW29.P0
- removed net D10: JP3.8, MOD1.PA6_A10_D10_MOSI
- removed net D2: JP3.5, MOD1.PA10_A2_D2
- removed net D3: JP3.7, MOD1.PA11_A3_D3
- removed net D8: JP3.12, MOD1.PA7_A8_D8_SCK
- removed net D9: JP3.10, MOD1.PA5_A9_D9_MISO
- removed net N$1: IC1.IO4_6, SW4.S
- removed net N$20: IC3.IO1_6, SW12.P0
- removed net N$25: IC3.IO1_5, SW24.P0
- removed net N$26: IC3.IO4_4, SW19.P0
- removed net N$32: IC3.IO3_0, SW22.P0
- removed net N$40: IC1.IO1_1, SW38.P0
- removed net N$41: IC1.IO0_2, SW28.P0
- removed net N$47: IC1.IO3_4, SW17.P0
- removed net N$48: IC1.IO2_0, SW50.P0
- removed net N$53: IC1.IO2_3, SW53.P0
- removed net N$54: IC3.IO3_5, SW33.P0
- removed net N$55: IC1.IO3_3, SW16.P0
- removed net N$6: IC3.IO0_6, SW9.P0
- removed net N$7: IC1.IO0_3, SW27.P0
- removed net N$74: IC3.IO4_6, SW43.P0
- removed net N$75: IC3.IO2_1, SW37.P0
- removed net N$78: IC3.IO3_6, SW45.P0
- removed net N$80: IC3.IO3_2, SW46.P0
- removed net N$82: IC3.IO2_5, SW47.P0
- removed net N$86: IC3.IO1_7, SW61.P0
- removed net SCL2: JP3.13, MOD1.PB09_A7_D7_RX, MOD4.SCL, R4.1
- removed net SDA2: JP3.14, MOD1.PB08_A6_D6_TX, MOD4.SDA, R3.1
- removed net VCC/2: C17.1, C22.1, CN2.TIP, IC3.A0, IC3.A1, IC3.VSS@1, IC3.VSS@2, IC3.VSS@3, IC3.VSS@4, IC3.VSS@5, IC3.VSS@6, J5.1, JP2.4
- removed net VIN: JP3.2, MOD1.5V
- new net +5V: CN3.P$6, CN4.P$6, JP5G$2.P$1, JP6G$6.P$1, MOD1.5V, SW1.VDD, SW13.VDD, SW14.VDD, SW15.VDD, SW16.VDD, SW17.VDD, SW18.VDD, SW2.VDD, SW25.VDD, SW26.VDD, SW27.VDD, SW28.VDD, SW29.VDD, SW30.VDD, SW37.VDD, SW38.VDD, SW39.VDD, SW40.VDD, SW41.VDD, SW42.VDD, SW49.VDD, SW50.VDD, SW51.VDD, SW52.VDD, SW53.VDD, SW54.VDD, SW58.VDD, SW59.VDD, SW60.VDD, SW61.VDD, SW62.VDD
- new net +5V/2: CN1.P$6, CN2.P$6, JP1G$2.P$1, JP2G$6.P$1, SW10.VDD, SW11.VDD, SW12.VDD, SW19.VDD, SW20.VDD, SW21.VDD, SW22.VDD, SW23.VDD, SW24.VDD, SW31.VDD, SW32.VDD, SW33.VDD, SW34.VDD, SW35.VDD, SW36.VDD, SW43.VDD, SW44.VDD, SW45.VDD, SW46.VDD, SW47.VDD, SW48.VDD, SW5.VDD, SW55.VDD, SW56.VDD, SW57.VDD, SW6.VDD, SW63.VDD, SW64.VDD, SW65.VDD, SW66.VDD, SW67.VDD, SW68.VDD, SW69_NICE.VDD, SW7.VDD, SW70.VDD, SW72.VDD, SW73.VDD, SW8.VDD, SW9.VDD
- new net COL10LED: SW15.DI, SW16.DO
- new net COL11LED: SW59.DI, SW60.DO
- new net COL12LED: SW17.DI, SW18.DO
- new net COL13LED: SW2.DO, SW62.DI
- new net COL1LED: SW72.DI, SW73.DO
- new net COL2LED: SW65.DI, SW7.DO
- new net COL3LED: SW5.DI, SW55.DO
- new net COL4LED: SW8.DI, SW9.DO
- new net COL5LED: SW46.DO, SW56.DI
- new net COL6LED: SW10.DI, SW11.DO
- new net COL7LED: SW57.DI, SW63.DO
- new net COL8LED: SW13.DI, SW14.DO
- new net COL9LED: SW50.DI, SW58.DO
- new net D6: MOD1.PB08_A6_D6_TX
- new net DISPLAY_BUSY: MOD1.PA5_A9_D9_MISO, X3-16.S
- new net DISPLAY_RESET: IC3.I/O1.7, R13.1, X3-15.S, X4-4.S
- new net EXPANDER0_INT: IC4.!INT, IC7A.I3, R7.1
- new net EXPANDER1_INT: IC2.!INT, IC7A.I4, R6.1
- new net EXPANDER2_INT: IC1.!INT, IC7A.I5, R5.1
- new net EXPANDER3_INT: IC5.!INT, IC6A.I5, R10.1
- new net EXPANDER4_INT: IC3.!INT, IC6A.I0, R3.1
- new net GDR: Q1.G, R9.2, X3-23.S
- new net INTERRUPT: IC6A.O, MOD1.PA11_A3_D3, R4.2
- new net LEFTER_HAND_INT: CN1.P$4, IC7A.I2, JP1G$4.P$1
- new net LEFTER_HAND_LED: CN1.P$3, JP1G$5.P$1, SW66.DO
- new net LEFT_HAND_INT: CN3.P$4, IC6A.I1, JP5G$4.P$1
- new net LEFT_HAND_INT': CN2.P$4, IC7A.O, JP2G$4.P$1, R14.2
- new net LEFT_HAND_LED: CN3.P$3, JP5G$5.P$1, SW61.DO
- new net LEFT_HAND_LED': CN2.P$3, JP2G$3.P$1, SW12.DI
- new net N$107: IC4.I/O1.5
- new net N$109: IC4.I/O1.7
- new net N$128: IC2.I/O0.0
- new net N$129: IC2.I/O0.1
- new net N$149: SW53.DO, SW60.DI
- new net N$150: SW41.DO, SW53.DI
- new net N$151: SW29.DO, SW41.DI
- new net N$152: SW17.DO, SW29.DI
- new net N$154: SW1.DO, SW2.DI
- new net N$163: SW15.DO, SW27.DI
- new net N$164: SW27.DO, SW39.DI
- new net N$165: SW39.DO, SW51.DI
- new net N$166: SW51.DO, SW58.DI
- new net N$18: SW11.DI, SW23.DO
- new net N$45: SW32.DO, SW44.DI
- new net N$58: SW6.DO, SW69_NICE.DI
- new net N$59: SW69_NICE.DO, SW73.DI
- new net N$61: IC4.I/O1.2
- new net N$62: IC4.I/O1.3
- new net N$65: SW64.DI, SW70.DO
- new net N$66: SW64.DO, SW66.DI
- new net PREVGH: C16.2, D1.C, X3-4.S
- new net PREVGL: C12.2, D3.A, X3-2.S
- new net QUAGSIRE: IC2.I/O0.2
- new net R0C0: IC4.I/O0.0, SW66.P0
- new net R0C1: IC4.I/O0.7, SW65.P1
- new net R0C10: IC5.I/O1.2, SW15.P0
- new net R0C11: IC5.I/O1.6, SW16.P1
- new net R0C12: IC3.I/O0.3, SW17.P0
- new net R0C13: IC3.I/O1.0, SW18.P0
- new net R0C2: IC2.I/O0.7, SW7.P1
- new net R0C3: IC2.I/O1.4, SW8.P1
- new net R0C4: IC1.I/O0.0, SW9.P1
- new net R0C5: IC1.I/O0.5, SW10.P1
- new net R0C6: IC1.I/O1.2, SW11.P1
- new net R0C7: IC1.I/O1.7, SW12.P1
- new net R0C8: IC5.I/O0.0, SW13.P0
- new net R0C9: IC5.I/O0.5, SW14.P0
- new net R1C0: IC4.I/O0.1, SW64.P0
- new net R1C1: IC4.I/O0.6, SW67.P1
- new net R1C10: IC5.I/O1.3, SW27.P0
- new net R1C11: IC5.I/O1.7, SW28.P0
- new net R1C12: IC3.I/O0.4, SW29.P0
- new net R1C13: IC3.I/O1.1, SW30.P0
- new net R1C2: IC2.I/O0.6, SW19.P1
- new net R1C3: IC2.I/O1.3, SW20.P1
- new net R1C4: IC2.I/O1.7, SW21.P1
- new net R1C5: IC1.I/O0.4, SW22.P1
- new net R1C6: IC1.I/O1.1, SW23.P1
- new net R1C7: IC1.I/O1.6, SW24.P1
- new net R1C8: IC5.I/O0.1, SW25.P0
- new net R1C9: IC5.I/O0.6, SW26.P0
- new net R2C0: IC4.I/O0.2, SW70.P0
- new net R2C1: IC4.I/O0.5, SW6.P1
- new net R2C10: IC5.I/O1.4, SW39.P0
- new net R2C11: IC3.I/O0.0, SW40.P0
- new net R2C12: IC3.I/O0.5, SW41.P0
- new net R2C13: IC3.I/O1.2, SW42.P0
- new net R2C2: IC2.I/O0.5, SW31.P1
- new net R2C3: IC2.I/O1.2, SW32.P1
- new net R2C4: IC2.I/O1.6, SW33.P1
- new net R2C5: IC1.I/O0.3, SW34.P1
- new net R2C6: IC1.I/O1.0, SW35.P1
- new net R2C7: IC1.I/O1.5, SW36.P1
- new net R2C8: IC5.I/O0.2, SW37.P0
- new net R2C9: IC5.I/O0.7, SW38.P0
- new net R3C0: IC4.I/O0.3, SW68.P0
- new net R3C1: IC4.I/O1.0, SW69_NICE.P0
- new net R3C10: IC5.I/O1.5, SW51.P0
- new net R3C11: IC3.I/O0.1, SW52.P0
- new net R3C12: IC3.I/O0.6, SW53.P0
- new net R3C13: IC3.I/O1.3, SW54.P0
- new net R3C2: IC2.I/O0.4, SW43.P1
- new net R3C3: IC2.I/O1.1, SW44.P1
- new net R3C4: IC2.I/O1.5, SW45.P1
- new net R3C5: IC1.I/O0.2, SW46.P1
- new net R3C6: IC1.I/O0.6, SW47.P1
- new net R3C7: IC1.I/O1.4, SW48.P1
- new net R3C8: IC5.I/O0.3, SW49.P0
- new net R3C9: IC5.I/O1.1, SW50.P0
- new net R4C0: IC4.I/O0.4, SW72.P0
- new net R4C1: IC4.I/O1.1, SW73.P0
- new net R4C10: IC5.I/O1.0, SW58.P1
- new net R4C11: IC3.I/O0.2, SW59.P0
- new net R4C12: IC3.I/O0.7, SW60.P0
- new net R4C13: IC3.I/O1.4, SW62.P0
- new net R4C14: IC3.I/O1.5, SW2.P1
- new net R4C15: IC3.I/O1.6, SW1.P0
- new net R4C2: IC2.I/O0.3, SW5.P1
- new net R4C3: IC2.I/O1.0, SW55.P1
- new net R4C4: IC1.I/O0.1, SW56.P0
- new net R4C6: IC1.I/O0.7, SW57.P0
- new net R4C7: IC1.I/O1.3, SW63.P1
- new net R4C8: IC5.I/O0.4, SW61.P0
- new net RAGE_LEDS: MOD1.PB09_A7_D7_RX, SW1.DI
- new net RESE: Q1.S, R11.2, X3-22.S
- new net RIGHTER_HAND_INT: CN4.P$4, IC6A.I6, JP6G$4.P$1
- new net RIGHTER_HAND_LED: CN4.P$3, JP6G$3.P$1, MOD1.PA10_A2_D2
- new net SCK: MOD1.PA7_A8_D8_SCK, X3-12.S
- new net SDI: MOD1.PA6_A10_D10_MOSI, X3-11.S
- new net THIRD_HALF_SELECT: IC1.A0, IC2.A0, IC4.A0, R8.1, SJ1.2, SJ2.2
- new net THIS_IS_LEFTER: IC4.I/O1.6, SJ2.1
- new net THIS_IS_RIGHTER: IC4.I/O1.4, SJ2.3
- new net TOUCH_INT: IC6A.I7, R12.1, X4-5.S
- new net TSCL: X3-19.S
- new net TSDA: X3-18.S
- new net VCCIO: C1.1, C19.1, C2.1, C3.1, CN1.P$7, CN2.P$7, IC1.A1, IC1.VDD, IC2.A1, IC2.A2, IC2.VDD, IC4.VDD, IC7P.VCC, JP1G$1.P$1, JP2G$7.P$1, R5.2, R6.2, R7.2, R8.2, SJ1.3
- new net VCOM: C13.2, X3-1.S
- new net VDD: C8.2, X3-7.S
- new net VGH: C15.2, X3-20.S
- new net VGL: C14.2, X3-21.S
- new net VPP: C9.2, X3-6.S
- new net VSH: C10.2, X3-5.S
- new net VSL: C11.2, X3-3.S
- net +3V3: now also C18.1, C4.1, C5.1, C6.1, C7.2, CN3.P$7, CN4.P$7, IC3.A0, IC3.A2, IC3.VDD, IC5.A2, IC5.VDD, IC6P.VCC, JP5G$1.P$1, JP6G$7.P$1, L1.1, R10.2, R12.2, R13.2, X3-10.S, X3-17.S, X3-9.S, X4-3.S; no longer C16.1, C3.1, CN1.TIP, IC1.A0, IC1.A1, IC1.A2, IC1.VSS@1, IC1.VSS@2, IC1.VSS@3, IC1.VSS@4, IC1.VSS@5, IC1.VSS@6, J5.2, JP1.1, JP3.6, MOD2.VCC, MOD3.VCC, MOD4.VCC, R4.2
- net D0: no longer JP3.1
- net D1: no longer JP3.3
- net GND: now also C10.1, C11.1, C12.1, C13.1, C14.1, C15.1, C16.1, C18.2, C4.2, C5.2, C6.2, C7.1, C8.1, C9.1, CN3.P$5, CN3.TABS, CN4.P$5, CN4.TABS, D2.C, IC3.A1, IC3.VSS, IC5.A0, IC5.A1, IC5.VSS, IC6P.GND, JP5G$3.P$1, JP6G$5.P$1, R11.1, R4.1, R9.1, SW1.GND, SW1.P1, SW13.GND, SW13.P1, SW14.GND, SW15.GND, SW16.GND, SW16.P0, SW17.GND, SW18.GND, SW2.GND, SW2.P0, SW25.GND, SW25.P1, SW26.GND, SW27.GND, SW28.GND, SW29.GND, SW30.GND, SW37.GND, SW37.P1, SW38.GND, SW39.GND, SW40.GND, SW41.GND, SW42.GND, SW49.GND, SW49.P1, SW50.GND, SW51.GND, SW52.GND, SW53.GND, SW54.GND, SW58.GND, SW58.P0, SW59.GND, SW60.GND, SW61.GND, SW61.P1, SW62.GND, X3-13.S, X3-14.S, X3-8.S, X4-6.S; no longer C16.2, C3.2, CN1.EARTH, IC1.!OE, IC1.VDD@1, IC1.VDD@2, J1.2, JP1.4, JP3.4, MOD2.GND, MOD3.GND, MOD4.GND, SW1.P, SW16.P1, SW2.P, SW3.P, SW4.P, SW5.P, SW58.P1, SW6.P
- net GND2: now also C1.2, C19.2, C2.2, C3.2, CN1.P$5, CN1.TABS, CN2.P$5, CN2.TABS, IC1.A2, IC1.VSS, IC2.VSS, IC4.A1, IC4.A2, IC4.VSS, IC7P.GND, JP1G$3.P$1, JP2G$5.P$1, R14.1, SJ1.1, SW10.GND, SW10.P0, SW11.GND, SW11.P0, SW12.GND, SW12.P0, SW19.GND, SW19.P0, SW20.GND, SW20.P0, SW21.GND, SW21.P0, SW22.GND, SW22.P0, SW23.GND, SW23.P0, SW24.GND, SW24.P0, SW31.GND, SW31.P0, SW32.GND, SW32.P0, SW33.GND, SW33.P0, SW34.GND, SW34.P0, SW35.GND, SW35.P0, SW36.GND, SW36.P0, SW43.GND, SW43.P0, SW44.GND, SW44.P0, SW45.GND, SW45.P0, SW46.GND, SW46.P0, SW47.GND, SW47.P0, SW48.GND, SW48.P0, SW5.GND, SW5.P0, SW55.GND, SW55.P0, SW56.GND, SW57.GND, SW6.GND, SW6.P0, SW63.GND, SW63.P0, SW64.GND, SW64.P1, SW65.GND, SW65.P0, SW66.GND, SW66.P1, SW67.GND, SW67.P0, SW68.GND, SW68.P1, SW69_NICE.GND, SW69_NICE.P1, SW7.GND, SW7.P0, SW70.GND, SW70.P1, SW72.GND, SW72.P1, SW73.GND, SW73.P1, SW8.GND, SW8.P0, SW9.GND, SW9.P0; no longer C17.2, C22.2, CN2.EARTH, IC3.!OE, IC3.A2, IC3.VDD@1, IC3.VDD@2, J1.1, JP2.1, SW10.P1, SW11.P1, SW12.P1, SW13.P1, SW19.P1, SW20.P1, SW21.P1, SW22.P1, SW23.P1, SW24.P1, SW25.P1, SW31.P1, SW32.P1, SW33.P1, SW34.P1, SW35.P1, SW36.P1, SW37.P1, SW43.P1, SW44.P1, SW45.P1, SW46.P1, SW47.P1, SW48.P1, SW49.P1, SW55.P1, SW61.P1, SW63.P1, SW7.P1, SW8.P1, SW9.P1
- net N$10: now also SW25.DO, SW37.DI; no longer IC1.IO1_7, SW58.P0
- net N$11: now also C17.1, D2.A, D3.C; no longer IC1.IO3_5, SW18.P0
- net N$12: now also SW35.DI, SW47.DO; no longer IC3.IO4_1, SW32.P0
- net N$13: now also SW37.DO, SW49.DI; no longer IC3.IO2_0, SW49.P0
- net N$14: now also SW23.DI, SW35.DO; no longer IC3.IO4_3, SW44.P0
- net N$15: now also SW42.DI, SW54.DO; no longer IC1.IO0_4, SW26.P0
- net N$16: now also SW54.DI, SW62.DO; no longer IC1.IO3_1, SW14.P0
- net N$17: now also C17.2, D1.A, L1.2, Q1.D; no longer IC1.IO0_0, SW30.P0
- net N$19: now also SW30.DI, SW42.DO; no longer IC3.IO2_7, SW57.P0
- net N$2: now also SW12.DO, SW24.DI; no longer IC3.IO4_2, SW7.P0
- net N$21: now also SW18.DI, SW30.DO; no longer IC3.IO3_7, SW56.P0
- net N$22: now also SW14.DI, SW26.DO; no longer IC1.IO1_2, SW54.P0
- net N$23: now also SW16.DI, SW28.DO; no longer IC3.IO4_7, SW55.P0
- net N$24: now also SW28.DI, SW40.DO; no longer IC1.IO0_5, SW42.P0
- net N$27: now also SW10.DO, SW22.DI; no longer IC1.IO3_6, SW1.S
- net N$28: now also SW22.DO, SW34.DI; no longer IC3.IO4_0, SW20.P0
- net N$29: now also SW40.DI, SW52.DO; no longer IC1.IO1_0, SW39.P0
- net N$3: now also SW24.DO, SW36.DI; no longer IC1.IO4_0, SW5.S
- net N$30: now also SW34.DO, SW46.DI; no longer IC3.IO3_4, SW21.P0
- net N$31: now also SW52.DI, SW59.DO; no longer IC1.IO1_5, SW62.P0
- net N$33: now also SW26.DI, SW38.DO; no longer IC1.IO0_7, SW40.P0
- net N$34: now also SW38.DI, SW50.DO; no longer IC3.IO2_3, SW13.P0
- net N$35: now also SW45.DI, SW56.DO; no longer IC3.IO1_4, SW36.P0
- net N$36: now also SW33.DI, SW45.DO; no longer IC3.IO1_0, SW35.P0
- net N$37: now also SW49.DO, SW61.DI; no longer IC1.IO1_3, SW60.P0
- net N$38: now also SW21.DI, SW33.DO; no longer IC3.IO1_3, SW48.P0
- net N$39: now also SW21.DO, SW9.DI; no longer IC1.IO1_6, SW59.P0
- net N$4: now also SW36.DO, SW48.DI; no longer IC3.IO0_5, SW8.P0
- net N$43: now also SW20.DI, SW8.DO; no longer IC3.IO1_1, SW23.P0
- net N$44: now also SW20.DO, SW32.DI; no longer IC3.IO1_2, SW11.P0
- net N$46: now also SW44.DO, SW55.DI; no longer IC1.IO4_7, SW6.S1
- net N$49: now also SW43.DI, SW5.DO; no longer IC1.IO2_1, SW51.P0
- net N$5: now also SW48.DO, SW63.DI; no longer IC1.IO4_5, SW2.S
- net N$50: now also SW31.DI, SW43.DO; no longer IC3.IO4_5, SW31.P0
- net N$51: now also SW19.DI, SW31.DO; no longer IC1.IO2_2, SW52.P0
- net N$52: now also SW19.DO, SW7.DI; no longer IC1.IO3_7, SW3.S
- net N$56: now also SW65.DO, SW67.DI; no longer IC3.IO3_1, SW34.P0
- net N$57: now also SW6.DI, SW67.DO; no longer IC3.IO2_6, SW63.P0
- net N$63: now also SW68.DI, SW72.DO; no longer IC1.IO3_2, SW15.P0
- net N$64: now also SW68.DO, SW70.DI; no longer IC1.IO0_6, SW41.P0
- net N$8: now also SW47.DI, SW57.DO; no longer IC3.IO0_7, SW10.P0
- net N$9: now also SW13.DO, SW25.DI; no longer IC3.IO2_2, SW25.P0
- net SCL: now also CN3.P$1, CN4.P$1, IC3.SCL, IC5.SCL, JP5G$7.P$1, JP6G$1.P$1, X4-2.S; no longer CN1.RING1, IC1.SCL, J3.2, JP1.2, JP3.11, MOD2.SCL, MOD3.SCL
- net SCL': now also CN1.P$1, CN2.P$1, IC1.SCL, IC2.SCL, IC4.SCL, JP1G$7.P$1, JP2G$1.P$1; no longer CN2.RING1, IC3.SCL, J3.1, JP2.3
- net SDA: now also CN3.P$2, CN4.P$2, IC3.SDA, IC5.SDA, JP5G$6.P$1, JP6G$2.P$1, X4-1.S; no longer CN1.RING2, IC1.SDA, J2.2, JP1.3, JP3.9, MOD2.SDA, MOD3.SDA
- net SDA': now also CN1.P$2, CN2.P$2, IC1.SDA, IC2.SDA, IC4.SDA, JP1G$6.P$1, JP2G$2.P$1; no longer CN2.RING2, IC3.SDA, J2.1, JP2.2
Other:
- note added: "+ LEDs (and rightest hand?) + Expander Interrupt + Expanders SDA/SCL + Touch SDA/SCL (same as expanders) + Touch interrupt X Rightest hand detect (Put on left hand board io expander) + Rightest hand LED + Display busy + Display reset X Display D/C (Not used - config for 3 wire SPI) X Display CS (Pull low) + Display SCK + Display SDI (MOSI)"
- note added: "All caps for eink must be 50V"
- note added: "BS"
- note added: "CSB"
- note added: "DC"
- note added: "Left half -->"
- note added: "Some keys, like this one, have reversed sockets to simplify routing"
- note added: "These are connected to an IO expander, which has built-in pullups. Feeding in third_half means this has no effect if this is the left half."
- note added: "Third half -->"
- note added: "This is actually TOUCH_RST! I ganged them to save GPIOs. -->"
- note removed: "These need pullups"
- note removed: "VSS and VDD are reversed"
- moved on the sheet: C16, C17, C3, R3, R4
